File: M252/M252.kicad_sch (KiCad schematic)
At the start: 16 parts, among them IC1 PIC16F1827-I/P, J101 UART, J102 PROG, J103 TRIP, Q5 10MHz, SW1 !MCLR

Commit message: v1.01 ガーバー出力
Parts:
- J102: footprint Connector_JST:JST_XH_B5B-XH-AM_1x05_P2.50mm_Vertical -> Connector_PinHeader_2.54mm:PinHeader_1x05_P2.54mm_Vertical
Other:
- note added: "To_RX (UNO 6pin)"
- note added: "To_TX (UNO 7pin)"
- note removed: "To_RX"
- note removed: "To_TX"
Changed lines of the file:
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@@
 	(title_block
 		(title "M252 TB2 adapter for M302")
-		(date "2024-12-08")
-		(rev "1.00")
+		(date "2024-12-10")
+		(rev "1.01")
 		(company "YS Lab")
 	)
@@
 		)
 	)
-	(text "To_TX"
-		(exclude_from_sim no)
-		(at 63.246 77.724 0)
+	(text "To_TX (UNO 7pin)"
+		(exclude_from_sim no)
+		(at 57.404 77.724 0)
 		(effects
 			(font
@@
 		)
 	)
-	(text "To_RX"
-		(exclude_from_sim no)
-		(at 63.5 80.01 0)
+	(text "To_RX (UNO 6pin)"
+		(exclude_from_sim no)
+		(at 57.15 80.01 0)
 		(effects
 			(font
@@
 			)
 		)
-		(property "Footprint" "Connector_JST:JST_XH_B5B-XH-AM_1x05_P2.50mm_Vertical"
+		(property "Footprint" "Connector_PinHeader_2.54mm:PinHeader_1x05_P2.54mm_Vertical"
 			(at 68.58 39.37 0)
 			(effects
@@
 			)
 		)
-		(property "Description" "Generic connector, single row, 01x05, script generated (kicad-library-utils/schlib/autogen/connector/)"
+		(property "Description" ""
 			(at 68.58 39.37 0)
 			(effects
