File: M252/M252.kicad_pcb (KiCad board)
At the start: 2 copper layers, 50 x 40 mm, 20 parts, among them IC101 PIC16F1827-I/P, J101 UART, J102 PROG, J103 TRIP, Q101 10MHz, SW101 !MCLR

Commit message: v1.01 ガーバー出力
Parts:
- J102: footprint Connector_JST:JST_XH_B5B-XH-AM_1x05_P2.50mm_Vertical -> Connector_PinHeader_2.54mm:PinHeader_1x05_P2.54mm_Vertical
- J103: footprint Connector_JST:JST_XH_B3B-XH-AM_1x03_P2.50mm_Vertical -> Connector_JST:JST_XH_B3B-XH-A_1x03_P2.50mm_Vertical
- turned J102 to -90 degrees
Routing:
- net Net-(J103-Pin_2): track 25.0 -> 33.8 mm
- net Net-(C104-Pad1): track 53.0 -> 49.2 mm
- net +5V: track 138.7 -> 136.5 mm
Other:
- board text added: "!MCLR"
- board text added: "PGC"
- board text added: "PGD"
- board text added: "V1.01"
- board text added: "VDD"
- board text removed: "V1.00"

Commit message: PCB発注前DRC済
Routing:
- net Net-(IC101-RB0): vias 0 -> 1
Changed lines of the file:
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@@
 		(tags "Resistor Axial_DIN0207 series Axial Horizontal pin pitch 7.62mm 0.25W = 1/4W length 6.3mm diameter 2.5mm")
 		(property "Reference" "R101"
-			(at -1.9812 0.0508 0)
+			(at 9.24 2.38 0)
 			(layer "F.SilkS")
 			(effects
@@
 		)
 		(property "Value" "22pF"
-			(at 1.23 -1.778 90)
+			(at 1.23 -1.936 90)
 			(layer "F.SilkS")
 			(effects
@@
 		(tags "connector JST XH vertical")
 		(property "Reference" "J103"
-			(at 2.5 -3.55 90)
+			(at 7.418 4.446 90)
 			(layer "F.SilkS")
 			(effects
@@
 	)
 	(segment
-		(start 112.776 79.629)
-		(end 116.459 79.629)
+		(start 124.206 66.04)
+		(end 124.206 71.628)
 		(width 0.2)
-		(layer "B.Cu")
+		(layer "F.Cu")
+		(net 11)
+	)
+	(segment
+		(start 117.856 73.5)
+		(end 117.856 65.786)
+		(width 0.2)
+		(layer "F.Cu")
 		(net 11)
 	)
@@
 		(end 124.206 66.04)
 		(width 0.2)
-		(layer "B.Cu")
+		(layer "F.Cu")
 		(net 11)
 	)
 	(segment
-		(start 118.872 64.77)
-		(end 122.936 64.77)
+		(start 117.856 65.786)
+		(end 118.872 64.77)
 		(width 0.2)
-		(layer "B.Cu")
+		(layer "F.Cu")
 		(net 11)
 	)
 	(segment
-		(start 124.206 66.04)
-		(end 124.206 71.628)
+		(start 118.872 64.77)
+		(end 122.936 64.77)
 		(width 0.2)
-		(layer "B.Cu")
+		(layer "F.Cu")
+		(net 11)
+	)
+	(via
+		(at 117.856 73.5)
+		(size 0.6)
+		(drill 0.3)
+		(layers "F.Cu" "B.Cu")
 		(net 11)
 	)
 	(segment
-		(start 117.856 78.232)
-		(end 117.856 65.786)
+		(start 117.856 73.5)
+		(end 117.856 78.232)
 		(width 0.2)
 		(layer "B.Cu")
@@
 	(segment
 		(start 116.459 79.629)
-		(end 117.856 78.232)
+		(end 112.776 79.629)
 		(width 0.2)
 		(layer "B.Cu")
@@
 	)
 	(segment
-		(start 117.856 65.786)
-		(end 118.872 64.77)
+		(start 117.856 78.232)
+		(end 116.459 79.629)
 		(width 0.2)
 		(layer "B.Cu")

Commit message: UNO直結タイプ1st
Parts:
- removed the REF** at (104.0, 96.0)
- removed the REF** at (104.0, 64.0)
- removed the REF** at (146.0, 64.0)
- removed the REF** at (146.0, 96.0)
- added REF**: Arduino_UNO_R3_WithMountingHoles, Module:Arduino_UNO_R3_WithMountingHoles, F.Cu at (115.2, 56.5)
- moved R101 29.6 mm to (108.2, 64.8), turned to -90 degrees
- moved R102 27.6 mm to (112.0, 72.4)
- moved C104 24.6 mm to (108.2, 61.4)
- moved R103 12.0 mm to (142.4, 66.0)
- moved R105 10.1 mm to (142.4, 91.4)
- moved J102 8.79 mm to (116.1, 98.0)
- moved J103 8.64 mm to (149.2, 86.0)
- moved C102 7.48 mm to (136.4, 76.8)
- moved C103 7.40 mm to (136.3, 72.0), turned to -90 degrees
- moved Q101 7.12 mm to (131.4, 72.0)
- moved SW101 6.70 mm to (102.2, 68.2)
- moved C101 5.75 mm to (146.8, 91.6), turned to 0 degrees
- moved C105 4.84 mm to (142.4, 69.8), turned to 180 degrees
- moved R104 4.40 mm to (142.4, 83.6)
- moved IC101 3.80 mm to (116.6, 67.0)
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Routing:
- net /TB2_TX: track 33.2 -> 105.5 mm, vias 0 -> 7
- net /TB2_RX: track 8.47 -> 70.9 mm, vias 0 -> 5
- net Net-(C104-Pad1): track 49.2 -> 12.1 mm
- net Net-(J103-Pin_2): track 33.8 -> 14.7 mm
- net Net-(IC101-RA5/~{MCLR}/VPP): track 54.8 -> 39.7 mm
- net Net-(IC101-RB6): track 22.6 -> 33.2 mm, vias 0 -> 1
- net +5V: track 136.5 -> 126.8 mm
- net Net-(IC101-RB7): track 23.5 -> 33.1 mm, vias 0 -> 2
- net Net-(IC101-RB0): track 31.0 -> 37.5 mm, vias 1 -> 0
- net Net-(IC101-RA6): track 15.3 -> 13.1 mm
- net Net-(IC101-RA7): track 12.8 -> 12.2 mm
Other:
- board size 50 x 40 mm -> 68.8 x 53.6 mm
- board text added: "TB2 adapter for Arduino UNO R3"
- board text added: "V2.00"
- board text removed: "TB2 adapter for M302"
- board text removed: "V1.01"
