File: M252VOLTERA/M252VOLTERA.kicad_pcb (KiCad board)
At the start: 2 copper layers, 50 x 40 mm, 20 parts, among them IC101 PIC16F1827-I/P, J101 UART, J102 PROG, J103 TRIP, Q101 10MHz, SW101 !MCLR

Commit message: VOLTERA Version
Parts:
- J101: footprint Connector_JST:JST_XH_B4B-XH-AM_1x04_P2.50mm_Vertical -> Connector_JST:JST_XH_B4B-XH-A_1x04_P2.50mm_Vertical
- moved SW101 0.80 mm to (106.5, 73.9)
Routing:
- net GND: track 18.5 -> 136.6 mm
- net Net-(IC101-RB7): track 23.5 -> 29.1 mm
- net Net-(IC101-RA4): track 47.9 -> 49.8 mm
- net Net-(C104-Pad1): track 57.3 -> 55.9 mm
- net Net-(J103-Pin_2): track 33.8 -> 33.2 mm
- net Net-(IC101-RB6): track 22.6 -> 22.0 mm
Other:
- board text added: "TB2 & M304K"
- board text added: "九州大学"
- board text removed: "Designed by YS-Lab. 2024"
- board text removed: "TB2 adapter for M302"
- board text removed: "V1.01"
- board text removed: "九州大学 AMPSD"
